File: tanmatsu.kicad_sch (KiCad schematic)
At the start: 47 parts, among them J1 USB device, J10 Headphone, J2 Expansion I3C, J3 SAO, J4 External Add-On (SAO / PMOD), J5 USB host, J6 CAMERA, J7 Internal Add-On, J8 Micro_SD_Card, J9 Speaker, SW1 Boot, U1 ESD, U2 ESD, U3 USBLC6-2P6, U4 TPD4E05U06DQAR, U5 CH334R, U6 USBLC6-2P6, Y1 12MHz

Commit message: Add ESD diode to headphone detect pin, add 1M pull-down resistor to SR latch (rev. 8)
Parts:
- removed C3: 10u, Capacitor_SMD:C_0805_2012Metric, symbol Device:C
- JP1: value ~ -> (none)
- renumbered C4 to C3
Connections:
- net at U5.15 (XO): now also Y1.1; no longer Y1.3
- net at U5.16 (XI): now also Y1.3; no longer Y1.1
Other:
- sheet Display ports: added SCL, SDA; removed none

Commit message: Add standoffs (Rev. 9)
Parts:
- H1, H2, H3, H4: footprint library:mountinghole_1.6mm -> library:SMTSO2030CTJ; LCSC - -> C2915626; now in the parts list
- H10, H11, H5, H6, H7, H8, H9: footprint MountingHole:MountingHole_2.2mm_M2_DIN965_Pad -> library:SMTSO2030CTJ; LCSC - -> C2915626; now in the parts list
Other:
- note added: "M2 holes for attaching back cover"
- note added: "M2 holes for attaching frontpanel"
- note removed: "1.6mm holes for attaching frontpanel"
- note removed: "M2 holes for expansion boards & case"
